Commit message: Update ROSCon_UK_2026 repo for ROS 2 Jazzy branch.

File: rosconuk26/urdf/irb120.urdf.xacro (robot description, xacro)
@@ -53,6 +53,5 @@
   <xacro:unless value="${bringup}">
     <gazebo>
-      <plugin filename="libgazebo_ros2_control.so" name="gazebo_ros2_control">
-        <robot_sim_type>gazebo_ros2_control/GazeboSystem</robot_sim_type>
+      <plugin filename="gz_ros2_control-system" name="gz_ros2_control::GazeboSimROS2ControlPlugin">
         <!-- IRB120 Controller -->
         <parameters>$(find ros2srrc_robots)/irb120/config/controller.yaml</parameters>

File: rosconuk26/urdf/rosconuk26_1.urdf.xacro (robot description, xacro)
@@ -53,6 +53,5 @@
   <xacro:unless value="${bringup}">
     <gazebo>
-      <plugin filename="libgazebo_ros2_control.so" name="gazebo_ros2_control">
-        <robot_sim_type>gazebo_ros2_control/GazeboSystem</robot_sim_type>
+      <plugin filename="gz_ros2_control-system" name="gz_ros2_control::GazeboSimROS2ControlPlugin">
         <!-- IRB120 Controller -->
         <parameters>$(find ros2srrc_robots)/irb120/config/controller.yaml</parameters>
@@ -73,10 +72,10 @@
       <origin xyz="0.0 0.0 0.0" rpy="0 0 0" />
       <geometry>
-        <mesh filename="file://$(find rosconuk26)/meshes/irb120enclosure/IRB120enclosure.dae" scale="1 1 1" />
+        <mesh filename="file://$(find rosconuk26)/meshes/irb120enclosure/IRB120enclosure.stl" scale="1 1 1" />
       </geometry>
     </collision>
     <inertial>
       <mass value="1000.0"/>
-      <inertia ixx="500.0" ixy="500.0" ixz="500.0" iyy="500.0" iyz="500.0" izz="500.0" />
+      <inertia ixx="200.0" ixy="0.0" ixz="0.0" iyy="200.0" iyz="0.0" izz="200.0"/>
     </inertial>
   </link>

File: rosconuk26/urdf/rosconuk26_2.urdf.xacro (robot description, xacro)
@@ -60,6 +60,5 @@
   <xacro:unless value="${bringup}">
     <gazebo>
-      <plugin filename="libgazebo_ros2_control.so" name="gazebo_ros2_control">
-        <robot_sim_type>gazebo_ros2_control/GazeboSystem</robot_sim_type>
+      <plugin filename="gz_ros2_control-system" name="gz_ros2_control::GazeboSimROS2ControlPlugin">
         <!-- IRB120 Controller -->
         <parameters>$(find ros2srrc_robots)/irb120/config/controller.yaml</parameters>
@@ -82,10 +81,10 @@
       <origin xyz="0.0 0.0 0.0" rpy="0 0 0" />
       <geometry>
-        <mesh filename="file://$(find rosconuk26)/meshes/irb120enclosure/IRB120enclosure.dae" scale="1 1 1" />
+        <mesh filename="file://$(find rosconuk26)/meshes/irb120enclosure/IRB120enclosure.stl" scale="1 1 1" />
       </geometry>
     </collision>
     <inertial>
       <mass value="1000.0"/>
-      <inertia ixx="500.0" ixy="500.0" ixz="500.0" iyy="500.0" iyz="500.0" izz="500.0" />
+      <inertia ixx="200.0" ixy="0.0" ixz="0.0" iyy="200.0" iyz="0.0" izz="200.0"/>
     </inertial>
   </link>
@@ -118,5 +117,5 @@
     <inertial>
       <mass value="10.0"/>
-      <inertia ixx="500.0" ixy="500.0" ixz="500.0" iyy="500.0" iyz="500.0" izz="500.0" />
+      <inertia ixx="200.0" ixy="0.0" ixz="0.0" iyy="200.0" iyz="0.0" izz="200.0"/>
     </inertial>
   </link>

File: rosconuk26/urdf/rosconuk26_3.urdf.xacro (robot description, xacro)
@@ -60,6 +60,5 @@
   <xacro:unless value="${bringup}">
     <gazebo>
-      <plugin filename="libgazebo_ros2_control.so" name="gazebo_ros2_control">
-        <robot_sim_type>gazebo_ros2_control/GazeboSystem</robot_sim_type>
+      <plugin filename="gz_ros2_control-system" name="gz_ros2_control::GazeboSimROS2ControlPlugin">
         <!-- IRB120 Controller -->
         <parameters>$(find ros2srrc_robots)/irb120/config/controller.yaml</parameters>
@@ -82,10 +81,10 @@
       <origin xyz="0.0 0.0 0.0" rpy="0 0 0" />
       <geometry>
-        <mesh filename="file://$(find rosconuk26)/meshes/irb120enclosure/IRB120enclosure.dae" scale="1 1 1" />
+        <mesh filename="file://$(find rosconuk26)/meshes/irb120enclosure/IRB120enclosure.stl" scale="1 1 1" />
       </geometry>
     </collision>
     <inertial>
       <mass value="1000.0"/>
-      <inertia ixx="500.0" ixy="500.0" ixz="500.0" iyy="500.0" iyz="500.0" izz="500.0" />
+      <inertia ixx="200.0" ixy="0.0" ixz="0.0" iyy="200.0" iyz="0.0" izz="200.0"/>
     </inertial>
   </link>
@@ -118,5 +117,5 @@
     <inertial>
       <mass value="10.0"/>
-      <inertia ixx="500.0" ixy="500.0" ixz="500.0" iyy="500.0" iyz="500.0" izz="500.0" />
+      <inertia ixx="200.0" ixy="0.0" ixz="0.0" iyy="200.0" iyz="0.0" izz="200.0"/>
     </inertial>
   </link>
@@ -137,13 +136,7 @@
         </geometry>
       </visual>
-      <collision>
-        <origin xyz="0.0 0.0 0.0" rpy="0 0 0" />
-        <geometry>
-          <mesh filename="file://$(find rosconuk26)/meshes/aruco/arucoGrid.dae" scale="1 1 1" />
-        </geometry>
-      </collision>
       <inertial>
         <mass value="10.0"/>
-        <inertia ixx="0.0002" ixy="0.0002" ixz="0.0002" iyy="0.0" iyz="0.0" izz="0.0" />
+        <inertia ixx="0.0002" ixy="0.0" ixz="0.0" iyy="0.0002" iyz="0.0" izz="0.0002" />
       </inertial>
     </link>
@@ -175,5 +168,5 @@
         <mass value="1.0" />
         <origin xyz="0 0 0" rpy="0 0 0"/>
-        <inertia ixx="0.0" ixy="0.0" ixz="0.0" iyy="0.0" iyz="0.0" izz="0.0" />
+        <inertia ixx="0.0005" ixy="0.0" ixz="0.0" iyy="0.0005" iyz="0.0" izz="0.0005"/>
       </inertial>
     </link>
@@ -184,6 +177,11 @@
     </joint>
     <gazebo reference="${prefix}camera_link">
-      <sensor name="camera" type="camera">
+      <sensor name="${prefix}camera" type="camera">
+        <pose>0 0 0 0 0 0</pose>
+        <always_on>true</always_on>
         <update_rate>30</update_rate>
+        <visualize>true</visualize>
+        <!-- Gz Transport topic -->
+        <topic>/camera/image_raw</topic>
         <camera name="head">
           <horizontal_fov>1.22</horizontal_fov>
@@ -193,24 +191,7 @@
             <format>R8G8B8</format>
           </image>
-          <clip>
-            <near>0.02</near>
-            <far>300</far>
-          </clip>
-          <noise>
-            <type>gaussian</type>
-            <mean>0.0</mean>
-            <stddev>0.007</stddev>
-          </noise>
+          <clip><near>0.02</near><far>300</far></clip>
+          <camera_info_topic>/camera/camera_info</camera_info_topic>
         </camera>
-        <plugin filename="libgazebo_ros_camera.so" name="camera_controller">
-          <robotNamespace/>
-          <alwaysOn>true</alwaysOn>
-          <updateRate>0.0</updateRate>
-          <cameraName>camera</cameraName>
-          <imageTopicName>image_raw</imageTopicName>
-          <cameraInfoTopicName>camera_info</cameraInfoTopicName>
-          <frameName>camera</frameName>
-          <hackBaseline>0.07</hackBaseline>
-        </plugin>
       </sensor>
     </gazebo>
