Commit message: Change object.urdf file naming.

File: rosconuk26/urdf/objects/RedCube.urdf (robot description, URDF)
Before this commit: robot cube, 1 links, 0 joints
Links:
- link ${name}: geometry collision mesh filename=file://$(find rosconuk26)/meshes/objects/RedCube.dae; visual mesh filename=file://$(find rosconuk26)/meshes/objects/RedCube.dae
